Commit message: fix robo model

File: my_amr_description/urdf/robot_structure.xacro (robot description, xacro)
@@ -91,5 +91,5 @@
         <parent link="base_link"/>
         <child link="right_wheel_link"/>
-        <axis xyz="0.0 -1.0 0.0"/>
+        <axis xyz="0.0 1.0 0.0"/>
     </joint>
     <joint name="base_left_wheel_joint" type="continuous">
